File: GPS + GSM Tracker with EEPROM Logging/GPS-GSM Tracker with EEPROM Logging.kicad_pcb (KiCad board)
At the start: 4 copper layers, 104 x 77.7 mm, 59 parts, among them J2 Conn_01x04_Pin, J4 Conn_01x02_Pin, J5 Conn_01x07_Pin, J6 Conn_01x04_Pin, J7 Conn_01x04_Pin, J8 Conn_01x07_Pin, J9 SIM_Card, SW1 SW_Push, SW2 SW_Push, U1 ESP32-S3-WROOM-1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

Commit message: Completed PCB design
Parts:
- added UART: UART, Connector_USB:USB_Micro-AB_Molex_47590-0001, F.Cu at (46.1, 62.2)
- added USB: USB, Connector_USB:USB_Micro-AB_Molex_47590-0001, F.Cu at (46.1, 73.0)
- J9: moved to B.Cu
- moved R27 12.1 mm to (62.7, 75.5)
- moved D13 12.0 mm to (66.3, 71.3)
- moved D14 12.0 mm to (62.7, 71.4)
- moved R28 11.8 mm to (66.2, 75.6)
- moved C14 11.3 mm to (69.1, 75.6)
- moved TH3 10.0 mm to (72.6, 76.1)
- turned J9 to 180 degrees
Connections:
- U1 pad 13: unconnected-(U1-USB_D--Pad13) -> Net-(J1-D-)
- U1 pad 14: unconnected-(U1-USB_D+-Pad14) -> Net-(J1-D+)
Routing:
- net /TX: track 41.5 -> 105.8 mm, vias 1 -> 2
- net /RX: track 41.0 -> 104.8 mm, vias 1 -> 2
- net Net-(J1-D-): track 0.00 -> 45.9 mm, vias 0 -> 2
- net GND: track 515.2 -> 560.1 mm, vias 15 -> 20
- net Net-(J1-D+): track 0.00 -> 44.1 mm, vias 0 -> 2
- net /BAT+(3.7V): track 102.0 -> 137.0 mm, vias 2 -> 4
- net Net-(U14-~{CHRG}): track 12.8 -> 22.5 mm
- net Net-(U14-~{STDBY}): track 12.3 -> 21.9 mm
- net Net-(U14-TEMP): track 17.4 -> 26.5 mm
- net /5V: track 87.4 -> 79.2 mm
- net Net-(J9-VCC): track 62.0 -> 55.9 mm, vias 2 -> 1
- net /3.3V: track 196.0 -> 198.1 mm, vias 4 -> 3
- net /TX1: track 67.2 -> 65.3 mm
- net /IO4: track 38.6 -> 39.4 mm
- net Net-(J9-CLK): track 44.7 -> 45.4 mm, vias 4 -> 2
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- added copper zone on In1.Cu, net /3.3V
- added copper zone on In2.Cu, net GND
Other:
- board size 104 x 77.7 mm -> 103.9 x 77.6 mm
- board text added: "GPS - GSM Tracking MCU - ESP32 S3 WROOM 1 Data collection with EEPROM 256kB"
- board text added: "KiCAD V9.0"
